File: kicad6/compara4/compara4.kicad_pcb (KiCad board)
At the start: 2 copper layers, 124 x 107.3 mm, 64 parts, among them J1 Conn_01x34_Female, J10 In_4, J11 CV_Jack, J12 Conn_02x05_Top_Bottom, J2 Conn_01x34_Male, J3 In_1, J4 In_2, J5 In_3, J6 Out_XOR, J7 Out_XNOR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

Commit message: compara4 layout tweaks
Routing:
- net GND: track 687.7 -> 685.1 mm
Changed lines of the file:
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@@
   (segment (start 180.34 124.46) (end 182.88 124.46) (width 1) (layer "B.Cu") (net 2))
   (segment (start 170.18 40.64) (end 162.56 40.64) (width 1) (layer "B.Cu") (net 2))
-  (segment (start 160.02 93.98) (end 160.025 93.975) (width 1) (layer "B.Cu") (net 2))
   (segment (start 114.3 71.12) (end 116.84 71.12) (width 1) (layer "B.Cu") (net 2))
   (segment (start 88.9 48.26) (end 88.9 45.72) (width 1) (layer "B.Cu") (net 2))
@@
   (segment (start 86.36 69.88) (end 86.36 71.12) (width 1) (layer "B.Cu") (net 2))
   (segment (start 71.12 71.12) (end 71.12 72.98) (width 1) (layer "B.Cu") (net 2))
+  (segment (start 170.18 99.06) (end 165.1 99.06) (width 1) (layer "B.Cu") (net 2))
   (segment (start 85.12 111.76) (end 86.36 110.52) (width 1) (layer "B.Cu") (net 2))
   (segment (start 86.36 71.12) (end 88.9 71.12) (width 1) (layer "B.Cu") (net 2))
-  (segment (start 157.48 93.98) (end 157.48 99.06) (width 1) (layer "B.Cu") (net 2))
   (segment (start 71.12 86.36) (end 78.74 86.36) (width 1) (layer "B.Cu") (net 2))
   (segment (start 120.65 40.64) (end 119.38 40.64) (width 1) (layer "B.Cu") (net 2))
@@
   (segment (start 180.34 124.46) (end 177.8 124.46) (width 1) (layer "B.Cu") (net 2))
   (segment (start 123.19 40.64) (end 121.92 40.64) (width 1) (layer "B.Cu") (net 2))
+  (segment (start 167.64 93.98) (end 167.64 99.06) (width 1) (layer "B.Cu") (net 2))
   (segment (start 88.9 48.26) (end 88.9 50.8) (width 0.25) (layer "B.Cu") (net 2))
   (segment (start 127 40.64) (end 123.19 40.64) (width 1) (layer "B.Cu") (net 2))
@@
   (segment (start 132.08 99.06) (end 147.32 99.06) (width 1) (layer "B.Cu") (net 2))
   (segment (start 132.08 124.46) (end 129.54 124.46) (width 1) (layer "B.Cu") (net 2))
-  (segment (start 160.02 93.98) (end 157.48 93.98) (width 1) (layer "B.Cu") (net 2))
   (segment (start 72.36 111.76) (end 71.12 110.52) (width 1) (layer "B.Cu") (net 2))
   (segment (start 129.54 127) (end 129.54 124.46) (width 1) (layer "B.Cu") (net 2))
@@
   (segment (start 177.8 129.54) (end 180.34 129.54) (width 1) (layer "B.Cu") (net 2))
   (segment (start 162.56 48.26) (end 162.56 40.64) (width 1) (layer "B.Cu") (net 2))
+  (segment (start 165.1 99.06) (end 157.48 99.06) (width 1) (layer "B.Cu") (net 2))
   (segment (start 147.32 99.06) (end 157.48 99.06) (width 1) (layer "B.Cu") (net 2))
   (segment (start 114.3 71.12) (end 111.76 71.12) (width 1) (layer "B.Cu") (net 2))
@@
   (segment (start 78.74 111.76) (end 72.36 111.76) (width 1) (layer "B.Cu") (net 2))
   (segment (start 180.3 71.12) (end 185.42 71.12) (width 1) (layer "B.Cu") (net 2))
-  (segment (start 170.18 99.06) (end 157.48 99.06) (width 1) (layer "B.Cu") (net 2))
   (segment (start 78.74 127) (end 71.12 127) (width 1) (layer "B.Cu") (net 2))
   (segment (start 121.92 124.46) (end 121.92 127) (width 1) (layer "B.Cu") (net 2))
@@
   (segment (start 157.48 76.2) (end 154.94 76.2) (width 1) (layer "B.Cu") (net 11))
   (segment (start 157.48 121.92) (end 149.86 121.92) (width 1) (layer "F.Cu") (net 12))
+  (segment (start 154.94 101.6) (end 154.94 96.52) (width 1) (layer "F.Cu") (net 12))
   (segment (start 157.48 101.6) (end 157.48 121.92) (width 1) (layer "F.Cu") (net 12))
-  (segment (start 153.67 96.52) (end 153.67 101.6) (width 1) (layer "F.Cu") (net 12))
   (via (at 157.48 101.6) (size 0.8) (drill 0.4) (layers "F.Cu" "B.Cu") (net 12))
-  (via (at 153.67 96.52) (size 0.8) (drill 0.4) (layers "F.Cu" "B.Cu") (net 12))
+  (via (at 154.94 96.52) (size 0.8) (drill 0.4) (layers "F.Cu" "B.Cu") (net 12))
   (via (at 149.855 121.925) (size 0.8) (drill 0.4) (layers "F.Cu" "B.Cu") (net 12))
-  (via (at 153.67 101.6) (size 0.8) (drill 0.4) (layers "F.Cu" "B.Cu") (net 12))
+  (via (at 154.94 101.6) (size 0.8) (drill 0.4) (layers "F.Cu" "B.Cu") (net 12))
+  (segment (start 152.4 96.52) (end 154.94 96.52) (width 1) (layer "B.Cu") (net 12))
   (segment (start 149.855 124.46) (end 149.855 121.925) (width 1) (layer "B.Cu") (net 12))
   (segment (start 142.24 119.38) (end 142.24 124.455) (width 1) (layer "B.Cu") (net 12))
@@
   (segment (start 142.24 96.52) (end 152.4 96.52) (width 1) (layer "B.Cu") (net 12))
   (segment (start 142.24 124.455) (end 142.235 124.46) (width 1) (layer "B.Cu") (net 12))
+  (segment (start 154.94 101.6) (end 180.34 101.6) (width 1) (layer "B.Cu") (net 12))
   (segment (start 147.31 119.38) (end 142.24 119.38) (width 1) (layer "B.Cu") (net 12))
   (segment (start 147.31 119.38) (end 149.86 119.38) (width 1) (layer "B.Cu") (net 12))
   (segment (start 180.34 99.06) (end 180.34 101.6) (width 1) (layer "B.Cu") (net 12))
-  (segment (start 153.67 101.6) (end 180.34 101.6) (width 1) (layer "B.Cu") (net 12))
-  (segment (start 152.4 96.52) (end 153.67 96.52) (width 1) (layer "B.Cu") (net 12))
   (segment (start 149.86 121.92) (end 149.855 121.925) (width 1) (layer "B.Cu") (net 12))
   (segment (start 179.07 86.36) (end 180.34 86.36) (width 1) (layer "B.Cu") (net 13))
